Commit message: Add aruco marker in scene

File: urdf/visual_servoing_scene.xacro (robot description, xacro)
@@ -119,3 +119,16 @@
         <child link="Yellow_marker"/>
     </joint>
+     <link name="ArucoMarker">
+        <visual>
+            <origin xyz="0 0 0" rpy="0 0 0"/>
+            <geometry>
+                <mesh filename="package://visual_servoing/meshes/marker2.dae" scale="1 1 1"/>
+            </geometry>
+        </visual>
+    </link>
+    <joint name="Markers_frame2ARUCO" type="fixed">
+        <origin xyz="0.3 0.3 0.3" rpy="-2.356 0 0"/>
+        <parent link="Markers_frame"/>
+        <child link="ArucoMarker"/>
+    </joint>
 </robot>
